Commit message: Stage 2: Robot model + FK, ros2_control backbone
- robot_model.py: ExcavatorModel with full FK chain, joint limits, base pose
- 19 unit tests for FK (zero config, swing, boom, stick, limits, base pose, SE3 validity)
- URDF updated with ros2_control block (mock_components/GenericSystem)
- excavator_control package: controller config (JointTrajectoryController + JSB)
- raw_urdf_publisher: workaround for robot_state_publisher stripping ros2_control tags
- excavator_control.launch.py: full stack launch with Foxglove Bridge
- All controllers load and activate successfully

File: excavator_description/urdf/excavator.urdf.xacro (robot description, xacro)
@@ -189,3 +189,42 @@
     <origin xyz="${bucket_length} 0 ${-bucket_depth}" rpy="0 0 0"/>
   </joint>
+  <!-- ===================== ros2_control ========================== -->
+  <ros2_control name="excavator_hw" type="system">
+    <hardware>
+      <plugin>mock_components/GenericSystem</plugin>
+      <param name="calculate_dynamics">false</param>
+    </hardware>
+    <!-- Cabin swing -->
+    <joint name="cabin_joint">
+      <command_interface name="position"/>
+      <state_interface name="position">
+        <param name="initial_value">0.0</param>
+      </state_interface>
+      <state_interface name="velocity"/>
+    </joint>
+    <!-- Boom -->
+    <joint name="boom_joint">
+      <command_interface name="position"/>
+      <state_interface name="position">
+        <param name="initial_value">0.0</param>
+      </state_interface>
+      <state_interface name="velocity"/>
+    </joint>
+    <!-- Stick -->
+    <joint name="stick_joint">
+      <command_interface name="position"/>
+      <state_interface name="position">
+        <param name="initial_value">0.0</param>
+      </state_interface>
+      <state_interface name="velocity"/>
+    </joint>
+    <!-- Bucket -->
+    <joint name="bucket_joint">
+      <command_interface name="position"/>
+      <state_interface name="position">
+        <param name="initial_value">0.0</param>
+      </state_interface>
+      <state_interface name="velocity"/>
+    </joint>
+  </ros2_control>
 </robot>

Commit message: Stage 3: Base motion planning
- base_planner.py: 3-phase trajectory (rotate-drive-rotate), BasePose, BaseTrajectory
- 23 unit tests for planner (goal reaching, sampling, error thresholds, wrap_angle)
- base_motion_node.py: executes trajectory, broadcasts world->base_link TF, publishes Path
- URDF: removed fixed world->base_link joint (now dynamic via base_motion_node)
- Both launch files updated to include base_motion_node
- Robot drives from (0,0,0) to working position (3,0,0) in 6 seconds

File: excavator_description/urdf/excavator.urdf.xacro (robot description, xacro)
@@ -37,7 +37,6 @@
     <color rgba="0.6 0.6 0.65 1.0"/>
   </material>
-  <!-- ===================== WORLD FRAME ========================== -->
-  <link name="world"/>
   <!-- ===================== BASE LINK ============================ -->
+  <!-- world → base_link transform is published dynamically by base_motion_node -->
   <link name="base_link">
     <visual>
@@ -60,10 +59,4 @@
     </inertial>
   </link>
-  <!-- Fixed joint from world to base (will be made movable later via ros2_control) -->
-  <joint name="base_joint" type="fixed">
-    <parent link="world"/>
-    <child  link="base_link"/>
-    <origin xyz="0 0 0" rpy="0 0 0"/>
-  </joint>
   <!-- ===================== CABIN (SWING) ======================== -->
   <link name="cabin_link">

Commit message: Improve joins

File: excavator_description/urdf/excavator.urdf.xacro (robot description, xacro)
@@ -17,7 +17,7 @@
   <xacro:property name="cabin_width"  value="1.0"/>
   <xacro:property name="cabin_height" value="0.8"/>
-  <xacro:property name="boom_length"  value="3.0"/>
+  <xacro:property name="boom_length"  value="3.5"/>
   <xacro:property name="boom_radius"  value="0.12"/>
-  <xacro:property name="stick_length" value="2.5"/>
+  <xacro:property name="stick_length" value="2.9"/>
   <xacro:property name="stick_radius" value="0.10"/>
   <xacro:property name="bucket_length" value="0.8"/>
@@ -114,5 +114,5 @@
     <origin xyz="${cabin_length} 0 ${cabin_height * 0.8}" rpy="0 0 0"/>
     <axis xyz="0 1 0"/>
-    <limit lower="-0.3" upper="1.2" effort="10000.0" velocity="0.5"/>
+    <limit lower="-0.5" upper="1.5" effort="10000.0" velocity="0.5"/>
     <dynamics damping="100.0" friction="20.0"/>
   </joint>
@@ -143,5 +143,5 @@
     <origin xyz="${boom_length} 0 0" rpy="0 0 0"/>
     <axis xyz="0 1 0"/>
-    <limit lower="-2.4" upper="0.0" effort="8000.0" velocity="0.5"/>
+    <limit lower="-2.7" upper="0.3" effort="8000.0" velocity="0.5"/>
     <dynamics damping="80.0" friction="15.0"/>
   </joint>
@@ -172,5 +172,5 @@
     <origin xyz="${stick_length} 0 0" rpy="0 0 0"/>
     <axis xyz="0 1 0"/>
-    <limit lower="-1.0" upper="2.2" effort="5000.0" velocity="0.8"/>
+    <limit lower="-1.5" upper="2.5" effort="5000.0" velocity="0.8"/>
     <dynamics damping="40.0" friction="10.0"/>
   </joint>

Commit message: Improvements

File: excavator_description/urdf/excavator.urdf.xacro (robot description, xacro)
@@ -143,5 +143,5 @@
     <origin xyz="${boom_length} 0 0" rpy="0 0 0"/>
     <axis xyz="0 1 0"/>
-    <limit lower="-2.7" upper="0.3" effort="8000.0" velocity="0.5"/>
+    <limit lower="-2.7" upper="2.7" effort="8000.0" velocity="0.5"/>
     <dynamics damping="80.0" friction="15.0"/>
   </joint>

Commit message: IMprove limits and make the markes update on position change

File: excavator_description/urdf/excavator.urdf.xacro (robot description, xacro)
@@ -114,5 +114,5 @@
     <origin xyz="${cabin_length} 0 ${cabin_height * 0.8}" rpy="0 0 0"/>
     <axis xyz="0 1 0"/>
-    <limit lower="-0.5" upper="1.5" effort="10000.0" velocity="0.5"/>
+    <limit lower="-1.5" upper="1.5" effort="10000.0" velocity="0.5"/>
     <dynamics damping="100.0" friction="20.0"/>
   </joint>
